Commit message: tunning left

File: quad_simulator/spot_description/spot.urdf (robot description, URDF)
Before this commit: robot spirit, 19 links, 18 joints
Links:
- removed link body_dummy
- removed link imu_link
- link body: mass 5.75 -> 16.70765207; geometry collision box size=0.85 0.24 0.18; visual mesh filename=package://spot_description/meshes/base_link_0_geom_visual_m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 scale=1 1 1
- link hip0: mass 0.575 -> 1.13688339; geometry visual mesh filename=package://spot_description/meshes/fl_hip_0_geom_visual_mesh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
- link hip1: mass 0.575 -> 1.13688339; geometry visual mesh filename=package://spot_description/meshes/hl_hip_0_geom_visual_mesh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
- link hip2: mass 0.575 -> 1.13688339; geometry visual mesh filename=package://spot_description/meshes/fr_hip_0_geom_visual_mesh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
- link hip3: mass 0.575 -> 1.13688339; geometry visual mesh filename=package://spot_description/meshes/hr_hip_0_geom_visual_mesh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
- link lower0: mass 0.075 -> 0.330; geometry collision cylinder length=0.03 radius=0.033; collision cylinder length=0.35 radius=0.015
- link lower1: mass 0.075 -> 0.330; geometry collision cylinder length=0.03 radius=0.033; collision cylinder length=0.35 radius=0.015
- link lower2: mass 0.075 -> 0.330; geometry collision cylinder length=0.03 radius=0.033; collision cylinder length=0.35 radius=0.015
- link lower3: mass 0.075 -> 0.330; geometry collision cylinder length=0.03 radius=0.033; collision cylinder length=0.35 radius=0.015
- link upper0: mass 0.775 -> 2.25620359; geometry collision cylinder length=0.35 radius=0.045; visual mesh filename=package://spot_description/meshes/l_uleg_0_geom_visual_mesh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
- link upper1: mass 0.775 -> 2.25620359; geometry collision cylinder length=0.35 radius=0.045; visual mesh filename=package://spot_description/meshes/l_uleg_0_geom_visual_mesh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
- link upper2: mass 0.775 -> 2.25620359; geometry collision cylinder length=0.35 radius=0.045; visual mesh filename=package://spot_description/meshes/r_uleg_0_geom_visual_mesh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
- link upper3: mass 0.775 -> 2.25620359; geometry collision cylinder length=0.35 radius=0.045; visual mesh filename=package://spot_description/meshes/r_uleg_0_geom_visual_mesh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
Joints:
- removed joint dummy_joint
- removed joint imu_joint
- joint 0: axis 0 -1 0 -> 0 1 0; limit lower=-6.28318530718 upper=6.28318530718 effort=40 velocity=30 -> lower=-0.89884456477707963539 upper=2.2951079663725435509 effort=1000 velocity=1000.00; origin xyz=0.0 0.10098 0 -> xyz=0.0 0.110945 0.0
- joint 1: limit lower=0 upper=3.14159265359 effort=40 velocity=30 -> lower=-2.7929 upper=-0.254402 effort=1000 velocity=1000.00; origin xyz=-0.206 0 0 -> xyz=0.025 0.000 -0.3205
- joint 10: limit lower=-0.707 upper=0.707 effort=40 velocity=30 -> lower=-0.78539816339744827899 upper=0.78539816339744827899 effort=1000 velocity=1000.00; origin xyz=0.2263 -0.07 0 -> xyz=0.29785 -0.05500 0.00000
- joint 11: limit lower=-0.707 upper=0.707 effort=40 velocity=30 -> lower=-0.78539816339744827899 upper=0.78539816339744827899 effort=1000 velocity=1000.00; origin xyz=-0.2263 -0.07 0 -> xyz=-0.29785 -0.05500 0.00000
- joint 2: axis 0 -1 0 -> 0 1 0; limit lower=-6.28318530718 upper=6.28318530718 effort=40 velocity=30 -> lower=-0.898845 upper=2.24363 effort=1000 velocity=1000.00; origin xyz=-0.0 0.10098 0 -> xyz=0.0 0.110945 0.0
- joint 3: limit lower=0 upper=3.14159265359 effort=40 velocity=30 -> lower=-2.7929 upper=-0.255648 effort=1000 velocity=1000.00; origin xyz=-0.206 0 0 -> xyz=0.025 0.000 -0.3205
- joint 4: axis 0 -1 0 -> 0 1 0; limit lower=-6.28318530718 upper=6.28318530718 effort=40 velocity=30 -> lower=-0.89884456477707963539 upper=2.2951079663725435509 effort=1000 velocity=1000.00; origin xyz=0.0 -0.10098 0 -> xyz=0.0 -0.110945 0.0
- joint 5: limit lower=0 upper=3.14159265359 effort=40 velocity=30 -> lower=-2.7929 upper=-0.247067 effort=1000 velocity=1000.00; origin xyz=-0.206 0 0 -> xyz=0.025 0.000 -0.3205
- joint 6: axis 0 -1 0 -> 0 1 0; limit lower=-6.28318530718 upper=6.28318530718 effort=40 velocity=30 -> lower=-0.89884456477707963539 upper=2.2951079663725435509 effort=1000 velocity=1000.00; origin xyz=-0.0 -0.10098 0 -> xyz=0.0 -0.110945 0.0
- joint 7: limit lower=0 upper=3.14159265359 effort=40 velocity=30 -> lower=-2.7929 upper=-0.248282 effort=1000 velocity=1000.00; origin xyz=-0.206 0 0 -> xyz=0.025 0.000 -0.3205
- joint 8: limit lower=-0.707 upper=0.707 effort=40 velocity=30 -> lower=-0.78539816339744827899 upper=0.78539816339744827899 effort=1000 velocity=1000.00; origin xyz=0.2263 0.07 0 -> xyz=0.29785 0.05500 0.00000
- joint 9: limit lower=-0.707 upper=0.707 effort=40 velocity=30 -> lower=-0.78539816339744827899 upper=0.78539816339744827899 effort=1000 velocity=1000.00; origin xyz=-0.2263 0.07 0 -> xyz=-0.29785 0.05500 0.00000
- joint jtoe0: origin xyz=0.206 0 -0.0 -> xyz=0 0 0
- joint jtoe1: origin xyz=0.206 0 -0.0 -> xyz=0 0 0.0
- joint jtoe2: origin xyz=0.206 0 -0.0 -> xyz=0 0 -0.0
- joint jtoe3: origin xyz=0.206 0 -0.0 -> xyz=0 0 -0.0

File: quad_simulator/spot_description/spot_og.urdf (robot description, URDF)
Before this commit: robot spirit, 19 links, 18 joints
Links:
- removed link body_dummy
- removed link imu_link
- link body: mass 5.75 -> 16.70765207; geometry collision box size=0.85 0.24 0.18; visual mesh filename=package://spot_description/meshes/base_link_0_geom_visual_m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
- link hip0: mass 0.575 -> 1.13688339; geometry visual mesh filename=package://spot_description/meshes/fl_hip_0_geom_visual_mesh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
- link hip1: mass 0.575 -> 1.13688339; geometry visual mesh filename=package://spot_description/meshes/hl_hip_0_geom_visual_mesh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
- link hip2: mass 0.575 -> 1.13688339; geometry visual mesh filename=package://spot_description/meshes/fr_hip_0_geom_visual_mesh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
- link hip3: mass 0.575 -> 1.13688339; geometry visual mesh filename=package://spot_description/meshes/hr_hip_0_geom_visual_mesh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
- link lower0: mass 0.075 -> 0.330; geometry collision cylinder length=0.03 radius=0.033; collision cylinder length=0.35 radius=0.015
- link lower1: mass 0.075 -> 0.330; geometry collision cylinder length=0.03 radius=0.033; collision cylinder length=0.35 radius=0.015
- link lower2: mass 0.075 -> 0.330; geometry collision cylinder length=0.03 radius=0.033; collision cylinder length=0.35 radius=0.015
- link lower3: mass 0.075 -> 0.330; geometry collision cylinder length=0.03 radius=0.033; collision cylinder length=0.35 radius=0.015
- link upper0: mass 0.775 -> 2.25620359; geometry collision cylinder length=0.35 radius=0.045; visual mesh filename=package://spot_description/meshes/l_uleg_0_geom_visual_mesh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
- link upper1: mass 0.775 -> 2.25620359; geometry collision cylinder length=0.35 radius=0.045; visual mesh filename=package://spot_description/meshes/l_uleg_0_geom_visual_mesh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
- link upper2: mass 0.775 -> 2.25620359; geometry collision cylinder length=0.35 radius=0.045; visual mesh filename=package://spot_description/meshes/r_uleg_0_geom_visual_mesh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
- link upper3: mass 0.775 -> 2.25620359; geometry collision cylinder length=0.35 radius=0.045; visual mesh filename=package://spot_description/meshes/r_uleg_0_geom_visual_mesh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
Joints:
- removed joint dummy_joint
- removed joint imu_joint
- joint 0: axis 0 -1 0 -> 0 1 0; limit lower=-6.28318530718 upper=6.28318530718 effort=40 velocity=30 -> lower=-0.89884456477707963539 upper=2.2951079663725435509 effort=1000 velocity=1000.00; origin xyz=0.0 0.10098 0 -> xyz=0.0 0.110945 0.0
- joint 1: limit lower=0 upper=3.14159265359 effort=40 velocity=30 -> lower=-2.7929 upper=-0.254402 effort=1000 velocity=1000.00; origin xyz=-0.206 0 0 -> xyz=0.025 0.000 -0.3205
- joint 10: limit lower=-0.707 upper=0.707 effort=40 velocity=30 -> lower=-0.78539816339744827899 upper=0.78539816339744827899 effort=1000 velocity=1000.00; origin xyz=0.2263 -0.07 0 -> xyz=0.29785 -0.05500 0.00000
- joint 11: limit lower=-0.707 upper=0.707 effort=40 velocity=30 -> lower=-0.78539816339744827899 upper=0.78539816339744827899 effort=1000 velocity=1000.00; origin xyz=-0.2263 -0.07 0 -> xyz=-0.29785 -0.05500 0.00000
- joint 2: axis 0 -1 0 -> 0 1 0; limit lower=-6.28318530718 upper=6.28318530718 effort=40 velocity=30 -> lower=-0.898845 upper=2.24363 effort=1000 velocity=1000.00; origin xyz=-0.0 0.10098 0 -> xyz=0.0 0.110945 0.0
- joint 3: limit lower=0 upper=3.14159265359 effort=40 velocity=30 -> lower=-2.7929 upper=-0.255648 effort=1000 velocity=1000.00; origin xyz=-0.206 0 0 -> xyz=0.025 0.000 -0.3205
- joint 4: axis 0 -1 0 -> 0 1 0; limit lower=-6.28318530718 upper=6.28318530718 effort=40 velocity=30 -> lower=-0.89884456477707963539 upper=2.2951079663725435509 effort=1000 velocity=1000.00; origin xyz=0.0 -0.10098 0 -> xyz=0.0 -0.110945 0.0
- joint 5: limit lower=0 upper=3.14159265359 effort=40 velocity=30 -> lower=-2.7929 upper=-0.247067 effort=1000 velocity=1000.00; origin xyz=-0.206 0 0 -> xyz=0.025 0.000 -0.3205
- joint 6: axis 0 -1 0 -> 0 1 0; limit lower=-6.28318530718 upper=6.28318530718 effort=40 velocity=30 -> lower=-0.89884456477707963539 upper=2.2951079663725435509 effort=1000 velocity=1000.00; origin xyz=-0.0 -0.10098 0 -> xyz=0.0 -0.110945 0.0
- joint 7: limit lower=0 upper=3.14159265359 effort=40 velocity=30 -> lower=-2.7929 upper=-0.248282 effort=1000 velocity=1000.00; origin xyz=-0.206 0 0 -> xyz=0.025 0.000 -0.3205
- joint 8: limit lower=-0.707 upper=0.707 effort=40 velocity=30 -> lower=-0.78539816339744827899 upper=0.78539816339744827899 effort=1000 velocity=1000.00; origin xyz=0.2263 0.07 0 -> xyz=0.29785 0.05500 0.00000
- joint 9: limit lower=-0.707 upper=0.707 effort=40 velocity=30 -> lower=-0.78539816339744827899 upper=0.78539816339744827899 effort=1000 velocity=1000.00; origin xyz=-0.2263 0.07 0 -> xyz=-0.29785 0.05500 0.00000
- joint jtoe0: origin xyz=0.206 0 -0.0 -> xyz=0 0 -0.0
- joint jtoe1: origin xyz=0.206 0 -0.0 -> xyz=0 0 -0.0
- joint jtoe2: origin xyz=0.206 0 -0.0 -> xyz=0 0 -0.0
- joint jtoe3: origin xyz=0.206 0 -0.0 -> xyz=0 0 -0.0
